File: SignalForgeV1.0.kicad_sch (KiCad schematic)
At the start: 49 parts, among them J1 USB_C_2.0, J2 BATTERY, J3 Micro_SD_Card_Det1, J4 Conn_01x03_Socket, Q1 DMG2301L, Q2 MMBT2222A, Q3 MMBT2222A, SW1 SW_Push, U1 LTC4054ES5-4.2, U2 CH340C, U3 PN5321A3HN_C1xx, U4 AP2112K-3.3, U6 ESP32-WROOM-32E

Commit message: feat: pcb design and 3d
Parts:
- removed C11, C12, C13, C15, C17, C18: 0.1uF, symbol Device:C_Small
- removed C14, C16: 10uF, symbol Device:C_Small
- removed FB1, FB2: FerriteBead_Small, symbol Device:FerriteBead_Small
- removed J1: USB_C_2.0, Connector_USB:USB_C_Receptacle_GCT_USB4105-xx-A_16P_TopMnt_Horizontal, symbol Connector:USB_C_Receptacle_USB2.0_16P
- removed J2: BATTERY, symbol Connector:Conn_01x02_Socket
- removed U3: PN5321A3HN_C1xx, Package_DFN_QFN:HVQFN-40-1EP_6x6mm_P0.5mm_EP4.1x4.1mm, symbol RF_NFC:PN5321A3HN_C1xx
- added AE1: Antenna, TestPoint:TestPoint_THTPad_D2.0mm_Drill1.0mm, symbol Device:Antenna
- added D3: IR Transmitter, LED_THT:LED_D5.0mm_Horizontal_O1.27mm_Z3.0mm, symbol Device:LED_Small_Filled
- added D4: LED_PWR, LED_SMD:LED_0805_2012Metric_Pad1.15x1.40mm_HandSolder, symbol Device:LED_Small_Filled
- added J1: PINOUT, Connector_PinSocket_2.54mm:PinSocket_1x08_P2.54mm_Horizontal, symbol Connector_Generic:Conn_01x08
- added J5: USB_B_Micro, Community:USB_B_Micro_SMD-TE, symbol Connector:USB_B_Micro
- added Q4: MMBT2222A, Package_TO_SOT_SMD:SOT-23, symbol Transistor_BJT:MMBT2222A
- added R14: 330R, Resistor_SMD:R_0805_2012Metric_Pad1.20x1.40mm_HandSolder, symbol Device:R_Small
- added R15, R23: 1k, Resistor_SMD:R_0805_2012Metric_Pad1.20x1.40mm_HandSolder, symbol Device:R_Small
- added R16, R17, R18, R19, R20, R21, R22: 10k, Resistor_SMD:R_0805_2012Metric_Pad1.20x1.40mm_HandSolder, symbol Device:R_Small
- added SW2: BACK_BTN, Button_Switch_SMD:SW_SPST_TL3342, symbol Switch:SW_Push
- added SW3: OK_BTN, Button_Switch_SMD:SW_SPST_TL3342, symbol Switch:SW_Push
- added SW4: UP_BTN, Button_Switch_SMD:SW_SPST_TL3342, symbol Switch:SW_Push
- added SW5: DOWN_BTN, Button_Switch_SMD:SW_SPST_TL3342, symbol Switch:SW_Push
- added SW6: RIGHT_BTN, Button_Switch_SMD:SW_SPST_TL3342, symbol Switch:SW_Push
- added SW7: LEFT_BTN, Button_Switch_SMD:SW_SPST_TL3342, symbol Switch:SW_Push
- added U3: ~, PN532_Module:PN532_Module, symbol PN532_Module:PN532_Module
- added U5: ~, SX1276_Module:SX1276_Module, symbol SX1276_Module:SX1276_Module
- added U7: 128x64, DM-OLED096-636:MODULE_DM-OLED096-636, symbol DM-OLED096-636:DM-OLED096-636
- BT1: footprint (none) -> Connector_JST:JST_EH_S2B-EH_1x02_P2.50mm_Horizontal
- C1, C10, C2, C3, C4, C5, C6, C7, C8, C9: footprint (none) -> Capacitor_SMD:C_0805_2012Metric_Pad1.18x1.45mm_HandSolder
- D2: footprint (none) -> LED_SMD:LED_0805_2012Metric_Pad1.15x1.40mm_HandSolder
- J3: footprint (none) -> Community:J_SD_Card-micro_socket_A
- J4: value Conn_01x03_Socket -> IR Receiver; footprint (none) -> Connector_PinHeader_2.54mm:PinHeader_1x03_P2.54mm_Vertical
- R1, R10, R11, R12, R13, R2, R3, R4, R5, R6, R7, R8, R9: footprint (none) -> Resistor_SMD:R_0805_2012Metric_Pad1.20x1.40mm_HandSolder
- SW1: footprint (none) -> Button_Switch_SMD:SW_SPST_EVQP7C
- U4: footprint Package_TO_SOT_SMD:SOT-23-5 -> Package_TO_SOT_SMD:SOT-23-5_HandSoldering
- U6: footprint RF_Module:ESP32-WROOM-32D -> RF_Module:ESP32-WROOM-32E
Connections:
- net +3V3: now also D3.2 (A), J1.4 (Pin_4), R16.1, R17.1, R18.1, R19.1, R20.1, R21.1, R22.1, R23.1, U3.1 (VCC), U5.5 (VCC), U7.1 (VCC_IN); no longer U2.4 (V3)
- net +BATT: now also BT1.1 (+), U1.3 (BAT)
- net D+: now also J5.3 (D+)
- net D-: now also J5.2 (D-)
- net GND: now also D4.1 (K), J1.3 (Pin_3), J5.5 (GND), J5.6 (Shield), R14.2, SW2.1, SW3.1, SW4.1, SW5.1, SW6.1, SW7.1, U3.2 (GND), U5.16 (GND), U5.2 (GND), U5.9 (GND), U7.2 (GND)
- net GPIO0: now also U6.25 (IO0)
- net IR_IN: now also R16.2
- net SD_CS: now also U6.29 (IO5)
- net VBUS: now also J5.1 (VBUS)
- net VSPI_MISO: now also U6.31 (IO19)
- net VSPI_MOSI: now also U6.37 (IO23)
- net VSPI_SCK: now also U6.30 (IO18)
- net VIN: now reaches C4.1, D1.1 (K), Q1.2 (S), R2.1, U4.1 (VIN)
- net LEFT_BTN: now reaches U6.10 (IO25)
- net LEFT_BTN: now also R22.2, SW7.2
- net DOWN_BTN: now reaches U6.11 (IO26)
- net DOWN_BTN: now also R20.2, SW5.2
- net UP_BTN: now reaches U6.12 (IO27)
- net UP_BTN: now also R19.2, SW4.2
- net HSPI_SCK: now reaches U6.13 (IO14)
- net HSPI_SCK: now also J1.8 (Pin_8), U5.12 (SCK)
- net HSPI_MISO: now reaches U6.14 (IO12)
- net HSPI_MISO: now also J1.7 (Pin_7), U5.10 (MISO)
- net HSPI_MOSI: now reaches U6.16 (IO13)
- net HSPI_MOSI: now also J1.6 (Pin_6), U5.11 (MOSI)
- net LORA_CS: now reaches U6.23 (IO15)
- net LORA_CS: now also U5.13 (NSS/CS)
- net NFC_IRQ: now reaches U6.26 (IO4)
- net NFC_IRQ: now also U3.9 (IRQ)
- net LORA_DI0: now reaches U6.27 (IO16)
- net LORA_DI0: now also U5.6 (DIO0)
- net BACK_BTN: now reaches U6.28 (IO17)
- net BACK_BTN: now also J1.5 (Pin_5), R17.2, SW2.2
- net SDA: now reaches U6.33 (IO21)
- net SDA: now also J1.1 (Pin_1), U3.3 (SDA), U7.4 (SDA)
- net SCL: now reaches U6.36 (IO22)
- net SCL: now also J1.2 (Pin_2), U3.4 (SCL), U7.3 (SCL)
- net RIGHT_BTN: now reaches U6.6 (IO34)
- net RIGHT_BTN: now also R21.2, SW6.2
- net OK_BTN: now reaches U6.8 (IO32)
- net OK_BTN: now also R18.2, SW3.2
- net IR_OUT: now reaches U6.9 (IO33)
- net IR_OUT: now also R15.1
- new net: AE1.1 (A), U5.1 (ANT)
- new net: Q4.1 (B), R15.2
- new net: Q4.2 (E), R14.1
- new net: D3.1 (K), Q4.3 (C)
- new net: D4.2 (A), R23.2
- no-connect marks 6 -> 21
Other:
- note added: "DISPLAY"
- note added: "IR Receiver 38KHz"
- note added: "IR Transmitter"
- note added: "LORA SX1276 (433-915MHz)"
- note added: "NFC / PN532 (13.56MHz)"
- note added: "PINOUT"
- note added: "USB-Micro-B to UART (CH340C)"
- note removed: "AVDD"
- note removed: "DVDD"
- note removed: "TVDD"
- note removed: "USB-C to UART (CH340C)"
- moved on the sheet: C1, C2, C3, C8, C9, J3, J4, Q2, Q3, R1, R10, R11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
